Commit message: Remove Gazebo simulation support

File: descriptions/my_dog/bw_description/urdf/robot.urdf (robot description, URDF)
Before this commit: robot bw, 19 links, 18 joints
Links:
- link FL_calf: geometry collision box size=0.175 0.018 0.026; visual mesh filename=file:///home/zbs/Desktop/ros2_q/install/bw_description/shar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 scale=1 1 1
- link FL_foot: geometry collision cylinder length=0.035 radius=0.099; visual mesh filename=file:///home/zbs/Desktop/ros2_q/install/bw_description/shar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
- link FL_hip: geometry collision cylinder length=0.13 radius=0.0395; visual mesh filename=file:///home/zbs/Desktop/ros2_q/install/bw_description/shar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 scale=1 1 1
- link FL_thigh: geometry collision box size=0.16 0.032 0.036; visual mesh filename=file:///home/zbs/Desktop/ros2_q/install/bw_description/shar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 scale=1 1 1
- link FR_calf: geometry collision box size=0.175 0.018 0.026; visual mesh filename=file:///home/zbs/Desktop/ros2_q/install/bw_description/shar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 scale=1 1 1
- link FR_foot: geometry collision cylinder length=0.035 radius=0.099; visual mesh filename=file:///home/zbs/Desktop/ros2_q/install/bw_description/shar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
- link FR_hip: geometry collision cylinder length=0.13 radius=0.0395; visual mesh filename=file:///home/zbs/Desktop/ros2_q/install/bw_description/shar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 scale=1 1 1
- link FR_thigh: geometry collision box size=0.16 0.032 0.036; visual mesh filename=file:///home/zbs/Desktop/ros2_q/install/bw_description/shar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 scale=1 1 1
- link RL_calf: geometry collision box size=0.175 0.018 0.026; visual mesh filename=file:///home/zbs/Desktop/ros2_q/install/bw_description/shar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 scale=1 1 1
- link RL_foot: geometry collision cylinder length=0.035 radius=0.099; visual mesh filename=file:///home/zbs/Desktop/ros2_q/install/bw_description/shar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
- link RL_hip: geometry collision cylinder length=0.13 radius=0.0395; visual mesh filename=file:///home/zbs/Desktop/ros2_q/install/bw_description/shar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 scale=1 1 1
- link RL_thigh: geometry collision box size=0.16 0.032 0.036; visual mesh filename=file:///home/zbs/Desktop/ros2_q/install/bw_description/shar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 scale=1 1 1
- link RR_calf: geometry collision box size=0.175 0.018 0.026; visual mesh filename=file:///home/zbs/Desktop/ros2_q/install/bw_description/shar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 scale=1 1 1
- link RR_foot: geometry collision cylinder length=0.035 radius=0.099; visual mesh filename=file:///home/zbs/Desktop/ros2_q/install/bw_description/shar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
- link RR_hip: geometry collision cylinder length=0.13 radius=0.0395; visual mesh filename=file:///home/zbs/Desktop/ros2_q/install/bw_description/shar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 scale=1 1 1
- link RR_thigh: geometry collision box size=0.16 0.032 0.036; visual mesh filename=file:///home/zbs/Desktop/ros2_q/install/bw_description/shar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 scale=1 1 1
- link trunk: geometry collision box size=0.3262 0.225 0.125; visual mesh filename=file:///home/zbs/Desktop/ros2_q/install/bw_description/shar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 scale=1 1 1

File: descriptions/my_dog/bw_description/xacro/leg.xacro (robot description, xacro)
@@ -142,21 +142,4 @@
       </inertial>
     </link>
-    <!-- 核心关节的gazebo配置 -->
-    <gazebo reference="${name}_hip">
-      <mu1>0.2</mu1>
-      <mu2>0.2</mu2>
-    </gazebo>
-    <gazebo reference="${name}_thigh">
-      <mu1>0.2</mu1>
-      <mu2>0.2</mu2>
-      <self_collide>0</self_collide>
-      <kp value="1000000.0"/>
-      <kd value="100.0"/>
-    </gazebo>
-    <gazebo reference="${name}_calf">
-      <mu1>0.6</mu1>
-      <mu2>0.6</mu2>
-      <self_collide>1</self_collide>
-    </gazebo>
     <!-- 核心关节的传动配置 -->
     <xacro:leg_core_transmission name="${name}"/>
@@ -204,12 +187,4 @@
       </inertial>
     </link>
-    <!-- 足部关节的gazebo配置 -->
-    <gazebo reference="${name}_foot">
-      <mu1>0.6</mu1>
-      <mu2>0.6</mu2>
-      <self_collide>1</self_collide>
-      <kp value="1000000.0"/>
-      <kd value="100.0"/>
-    </gazebo>
     <!-- 足部关节的传动配置 -->
     <xacro:leg_foot_transmission name="${name}"/>

File: descriptions/my_dog/bw_description/xacro/robot.xacro (robot description, xacro)
@@ -2,20 +2,8 @@
 <robot name="bw" xmlns:xacro="http://www.ros.org/wiki/xacro">
   <xacro:arg name="DEBUG" default="false"/>
-  <xacro:arg name="GAZEBO" default="false"/>
-  <xacro:arg name="CLASSIC" default="false"/>
   <xacro:include filename="$(find bw_description)/xacro/const.xacro"/>
   <xacro:include filename="$(find bw_description)/xacro/materials.xacro"/>
   <xacro:include filename="$(find bw_description)/xacro/leg.xacro"/>
-  <xacro:if value="$(arg GAZEBO)">
-    <xacro:if value="$(arg CLASSIC)">
-      <xacro:include filename="$(find bw_description)/xacro/gazebo_classic.xacro"/>
-    </xacro:if>
-    <xacro:unless value="$(arg CLASSIC)">
-      <xacro:include filename="$(find bw_description)/xacro/gazebo.xacro"/>
-    </xacro:unless>
-  </xacro:if>
-  <xacro:unless value="$(arg GAZEBO)">
-    <xacro:include filename="$(find bw_description)/xacro/ros2_control.xacro"/>
-  </xacro:unless>
+  <xacro:include filename="$(find bw_description)/xacro/ros2_control.xacro"/>
   <!-- <xacro:stairs stairs="15" xpos="0" ypos="0" zpos="0" /> -->
   <!-- Rotor related joint and link is only for demonstrate location. -->
